File: Penguino-4260-Hardware/Penguino-Feather-4260-v1.2/Penguino-Feather-4260-v1.kicad_pcb (KiCad board)
At the start: 4 copper layers, 22.9 x 50.8 mm, 60 parts, among them J1 U.FL-R-SMT-1, J2 SMA-Edge-Mount, J3 USB_C_Receptacle_USB2.0, J4 JST_PH, J5 Conn_ARM_JTAG_SWD_10, Q1 SI2323DS, SW1 USR_BTN, SW2 RESET, U1 MCP73831, U2 ME6215C33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

Commit message: sch, pcb: v1.2 updates
Parts:
- removed REF**: OSHW-Symbol_6.7x6mm_SilkScreen, Symbol:OSHW-Symbol_6.7x6mm_SilkScreen
- added JP5: USB_P, Jumper:SolderJumper-3_P1.3mm_Bridged12_Pad1.0x1.5mm, B.Cu at (137.7, 76.7)
- added JP6: USB_N, Jumper:SolderJumper-3_P1.3mm_Bridged12_Pad1.0x1.5mm, B.Cu at (134.1, 76.7)
- added JP7: UART_VCC, Jumper:SolderJumper-2_P1.3mm_Bridged_RoundedPad1.0x1.5mm, B.Cu at (140.8, 87.5)
- added JP8: Rx, Jumper:SolderJumper-2_P1.3mm_Bridged_RoundedPad1.0x1.5mm, B.Cu at (129.5, 106.9)
- added JP9: Tx, Jumper:SolderJumper-2_P1.3mm_Bridged_RoundedPad1.0x1.5mm, B.Cu at (129.5, 109.1)
- added U9: CH340E, Package_SO:MSOP-10_3x3mm_P0.5mm, B.Cu at (141.6, 79.5)
- C6: value DNM -> 100nF; footprint Capacitor_SMD:C_0402_1005Metric -> Capacitor_SMD:C_0603_1608Metric; moved to B.Cu
- moved C6 35.0 mm to (143.8, 79.5), turned to 270 degrees
- moved G*** 11.1 mm to (131.5, 86.6)
- moved D3 0.13 mm to (134.9, 112.5)
Connections:
- C6 pad 1: Net-(C5-Pad2) -> GND
- C6 pad 2: GND -> Net-(C6-Pad2)
- U4 pad 26: USB_P -> MCU_U_P
- U4 pad 27: USB_N -> MCU_U_N
Routing:
- net Net-(JP9-Pad2): track 0.00 -> 35.9 mm
- net Net-(JP8-Pad2): track 0.00 -> 35.2 mm
- net MCU_U_P: track 0.00 -> 22.8 mm, vias 0 -> 1
- net MCU_U_N: track 0.00 -> 22.8 mm, vias 0 -> 1
- net USB_N: track 29.8 -> 8.53 mm, vias 4 -> 3
- net USB_P: track 30.5 -> 9.27 mm, vias 2 -> 1
- net Net-(C6-Pad2): track 0.00 -> 11.5 mm
- net /UD-: track 0.00 -> 9.37 mm
- net /UD+: track 0.00 -> 8.12 mm
- net GND: track 67.6 -> 74.0 mm, vias 115 -> 125
- net +3V3: track 65.8 -> 71.4 mm
- net PA04_TX1: track 9.24 -> 13.0 mm
- net PA05_RX1: track 5.59 -> 9.17 mm
Other:
- board text added: "v1.2"
- board text removed: "open hardware"
- board text removed: "v1.1"
