File: Penguino-4260-Hardware/Penguino-Feather-4260-v1.2/Penguino-Feather-4260-v1.sch (KiCad schematic (older format))
At the start: 57 parts, among them J1 U.FL-R-SMT-1, J2 SMA-Edge-Mount, J3 USB_C_Receptacle_USB2.0, J4 JST_PH, J5 Conn_ARM_JTAG_SWD_10, Q1 SI2323DS, SW1 USR_BTN, SW2 RESET, U1 MCP73831, U2 ME6215C33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

Commit message: sch, pcb: v1.2 updates
Parts:
- removed C6: DNM, Capacitor_SMD:C_0402_1005Metric, symbol Device:C_Small
- added C6: 100nF, Capacitor_SMD:C_0603_1608Metric, symbol Device:C
- added JP5: USB_P, Jumper:SolderJumper-3_P1.3mm_Bridged12_Pad1.0x1.5mm, symbol Jumper:SolderJumper_3_Bridged12
- added JP6: USB_N, Jumper:SolderJumper-3_P1.3mm_Bridged12_Pad1.0x1.5mm, symbol Jumper:SolderJumper_3_Bridged12
- added JP7: UART_VCC, Jumper:SolderJumper-2_P1.3mm_Bridged_RoundedPad1.0x1.5mm, symbol Jumper:SolderJumper_2_Bridged
- added JP8: Rx, Jumper:SolderJumper-2_P1.3mm_Bridged_RoundedPad1.0x1.5mm, symbol Jumper:SolderJumper_2_Bridged
- added JP9: Tx, Jumper:SolderJumper-2_P1.3mm_Bridged_RoundedPad1.0x1.5mm, symbol Jumper:SolderJumper_2_Bridged
- added U9: CH340E, Package_SO:MSOP-10_3x3mm_P0.5mm, symbol Interface_USB:CH340E
- J3: symbol Connector:USB_C_Receptacle_USB2.0 -> Penguino-Feather-4260-v1-rescue:USB_C_Receptacle_USB2.0-Connector
- U4: symbol rak4260:RAK4260 -> Penguino-Feather-4260-v1-rescue:RAK4260-rak4260
Connections:
- net labels added: MCU_U_N, MCU_U_P, UD+, UD-
- wire segments 257 -> 279
- no-connect marks 7 -> 10
Other:
- note added: "4.5V max.!"
- moved on the sheet: J4, J5, R13, R14, R17, U7, U8
